File: pcb/bled-stamp/power.kicad_sch (KiCad schematic)
At the start: 34 parts, among them SW6 SW_Push, U3 BQ25895RTWR, U4 TLV62595DMQR

Commit message: wip
Parts:
- U4: footprint DMQ0006A-MFG -> bled:DMQ0006A-MFG
Connections:
- net GND: now also U3.25 (PAD)
- net PMID renamed +5V
Other:
- moved on the sheet: C25
Changed lines of the file:
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@@
 	)
 	(junction
-		(at 53.34 53.34)
-		(diameter 0)
-		(color 0 0 0 0)
-	)
-	(junction
 		(at 76.2 167.64)
 		(diameter 0)
@@
 	)
 	(junction
+		(at 99.06 119.38)
+		(diameter 0)
+		(color 0 0 0 0)
+	)
+	(junction
 		(at 241.3 46.99)
 		(diameter 0)
@@
 	)
 	(junction
+		(at 53.34 58.42)
+		(diameter 0)
+		(color 0 0 0 0)
+	)
+	(junction
 		(at 31.75 114.3)
 		(diameter 0)
@@
 	(wire
 		(pts
+			(xy 44.45 66.04) (xy 55.88 66.04)
+		)
+		(stroke
+			(width 0)
+			(type default)
+		)
+	)
+	(wire
+		(pts
 			(xy 97.79 88.9) (xy 97.79 91.44)
 		)
@@
 	(wire
 		(pts
-			(xy 53.34 53.34) (xy 53.34 58.42)
+			(xy 53.34 50.8) (xy 53.34 58.42)
 		)
 		(stroke
@@
 	(wire
 		(pts
-			(xy 53.34 50.8) (xy 53.34 53.34)
+			(xy 99.06 119.38) (xy 99.06 121.92)
 		)
 		(stroke
@@
 	(wire
 		(pts
-			(xy 96.52 109.22) (xy 114.3 109.22)
+			(xy 44.45 50.8) (xy 44.45 66.04)
 		)
 		(stroke
@@
 	(wire
 		(pts
-			(xy 96.52 68.58) (xy 97.79 68.58)
+			(xy 96.52 109.22) (xy 114.3 109.22)
 		)
 		(stroke
@@
 	(wire
 		(pts
-			(xy 57.15 166.37) (xy 57.15 167.64)
+			(xy 96.52 68.58) (xy 97.79 68.58)
 		)
 		(stroke
@@
 	(wire
 		(pts
-			(xy 50.8 175.26) (xy 57.15 175.26)
+			(xy 57.15 166.37) (xy 57.15 167.64)
 		)
 		(stroke
@@
 	(wire
 		(pts
-			(xy 254 46.99) (xy 266.7 46.99)
+			(xy 50.8 175.26) (xy 57.15 175.26)
 		)
 		(stroke
@@
 	(wire
 		(pts
-			(xy 209.55 54.61) (xy 209.55 57.15)
+			(xy 254 46.99) (xy 266.7 46.99)
 		)
 		(stroke
@@
 	(wire
 		(pts
-			(xy 53.34 109.22) (xy 55.88 109.22)
+			(xy 209.55 54.61) (xy 209.55 57.15)
 		)
 		(stroke
@@
 	(wire
 		(pts
-			(xy 99.06 116.84) (xy 99.06 121.92)
+			(xy 53.34 109.22) (xy 55.88 109.22)
 		)
 		(stroke
@@
 	(wire
 		(pts
-			(xy 38.1 53.34) (xy 53.34 53.34)
+			(xy 99.06 116.84) (xy 99.06 119.38)
 		)
 		(stroke
@@
 	(wire
 		(pts
-			(xy 53.34 66.04) (xy 55.88 66.04)
-		)
-		(stroke
-			(width 0)
-			(type default)
-		)
-	)
-	(wire
-		(pts
 			(xy 195.58 57.15) (xy 198.12 57.15)
 		)
@@
 	(wire
 		(pts
+			(xy 25.4 58.42) (xy 53.34 58.42)
+		)
+		(stroke
+			(width 0)
+			(type default)
+		)
+	)
+	(wire
+		(pts
 			(xy 203.2 57.15) (xy 209.55 57.15)
 		)
@@
 	(wire
 		(pts
+			(xy 96.52 119.38) (xy 99.06 119.38)
+		)
+		(stroke
+			(width 0)
+			(type default)
+		)
+	)
+	(wire
+		(pts
 			(xy 97.79 73.66) (xy 118.11 73.66)
 		)
@@
 		)
 	)
-	(label "PMID"
-		(at 57.15 166.37 90)
-		(effects
-			(font
-				(size 1.27 1.27)
-			)
-			(justify left bottom)
-		)
-	)
-	(label "PMID"
-		(at 53.34 66.04 180)
-		(effects
-			(font
-				(size 1.27 1.27)
-			)
-			(justify right bottom)
-		)
-	)
 	(label "STAT"
 		(at 127 167.64 90)
@@
 	)
 	(symbol
+		(lib_id "power:+5V")
+		(at 44.45 50.8 0)
+		(unit 1)
+		(body_style 1)
+		(exclude_from_sim no)
+		(in_bom yes)
+		(on_board yes)
+		(in_pos_files yes)
+		(dnp no)
+		(fields_autoplaced yes)
+		(property "Reference" "#PWR095"
+			(at 44.45 54.61 0)
+			(hide yes)
+			(show_name no)
+			(do_not_autoplace no)
+			(effects
+				(font
+					(size 1.27 1.27)
+				)
+			)
+		)
+		(property "Value" "+5V"
+			(at 44.45 45.72 0)
+			(show_name no)
+			(do_not_autoplace no)
+			(effects
+				(font
+					(size 1.27 1.27)
+				)
+			)
+		)
+		(property "Footprint" ""
+			(at 44.45 50.8 0)
+			(hide yes)
+			(show_name no)
+			(do_not_autoplace no)
+			(effects
+				(font
+					(size 1.27 1.27)
+				)
+			)
+		)
+		(property "Datasheet" ""
+			(at 44.45 50.8 0)
+			(hide yes)
+			(show_name no)
+			(do_not_autoplace no)
+			(effects
+				(font
+					(size 1.27 1.27)
+				)
+			)
+		)
+		(property "Description" "Power symbol creates a global label with name \"+5V\""
+			(at 44.45 50.8 0)
+			(hide yes)
+			(show_name no)
+			(do_not_autoplace no)
+			(effects
+				(font
+					(size 1.27 1.27)
+				)
+			)
+		)
+		(pin "1"
+		)
+		(instances
+			(project "bled-stamp"
+				(path "/e988e766-358b-4d27-8746-3fe94b603f13"
+					(reference "#PWR095")
+					(unit 1)
+				)
+			)
+		)
+	)
+	(symbol
 		(lib_id "Device:C")
 		(at 63.5 171.45 0)
@@
 			)
 		)
-		(property "Footprint" "DMQ0006A-MFG"
+		(property "Footprint" "bled:DMQ0006A-MFG"
 			(at 177.8 50.8 0)
 			(hide yes)
@@
 	(symbol
 		(lib_id "Device:C")
-		(at 38.1 57.15 0)
+		(at 25.4 62.23 0)
 		(unit 1)
 		(body_style 1)
@@
 		(fields_autoplaced yes)
 		(property "Reference" "C25"
-			(at 41.91 55.8799 0)
+			(at 29.21 60.9599 0)
 			(show_name no)
 			(do_not_autoplace no)
@@
 		)
 		(property "Value" "1u"
-			(at 41.91 58.4199 0)
+			(at 29.21 63.4999 0)
 			(show_name no)
 			(do_not_autoplace no)
@@
 		)
 		(property "Footprint" ""
-			(at 39.0652 60.96 0)
+			(at 26.3652 66.04 0)
 			(hide yes)
 			(show_name no)
@@
 		)
 		(property "Datasheet" ""
-			(at 38.1 57.15 0)
+			(at 25.4 62.23 0)
 			(hide yes)
 			(show_name no)
@@
 		)
 		(property "Description" "Unpolarized capacitor"
-			(at 38.1 57.15 0)
+			(at 25.4 62.23 0)
 			(hide yes)
 			(show_name no)
@@
 	(symbol
 		(lib_id "power:GND")
-		(at 38.1 60.96 0)
+		(at 25.4 66.04 0)
 		(unit 1)
 		(body_style 1)
@@
 		(fields_autoplaced yes)
 		(property "Reference" "#PWR075"
-			(at 38.1 67.31 0)
+			(at 25.4 72.39 0)
 			(hide yes)
 			(show_name no)
@@
 		)
 		(property "Value" "GND"
-			(at 38.1 66.04 0)
+			(at 25.4 71.12 0)
 			(show_name no)
 			(do_not_autoplace no)
@@
 		)
 		(property "Footprint" ""
-			(at 38.1 60.96 0)
+			(at 25.4 66.04 0)
 			(hide yes)
 			(show_name no)
@@
 		)
 		(property "Datasheet" ""
-			(at 38.1 60.96 0)
+			(at 25.4 66.04 0)
 			(hide yes)
 			(show_name no)
@@
 		)
 		(property "Description" "Power symbol creates a global label with name \"GND\" , ground"
-			(at 38.1 60.96 0)
+			(at 25.4 66.04 0)
 			(hide yes)
 			(show_name no)
@@
 					(unit 1)
 				)
+			)
+		)
+	)
+	(symbol
+		(lib_id "power:+5V")
+		(at 57.15 166.37 0)
+		(unit 1)
+		(body_style 1)
+		(exclude_from_sim no)
+		(in_bom yes)
+		(on_board yes)
+		(in_pos_files yes)
+		(dnp no)
+		(fields_autoplaced yes)
+		(property "Reference" "#PWR096"
+			(at 57.15 170.18 0)
+			(hide yes)
+			(show_name no)
+			(do_not_autoplace no)
+			(effects
+				(font
+					(size 1.27 1.27)
+				)
+			)
+		)
+		(property "Value" "+5V"
+			(at 57.15 161.29 0)
+			(show_name no)
+			(do_not_autoplace no)
+			(effects
+				(font
+					(size 1.27 1.27)
+				)
+			)
+		)
+		(property "Footprint" ""
+			(at 57.15 166.37 0)
+			(hide yes)
+			(show_name no)
+			(do_not_autoplace no)
+			(effects
+				(font
+					(size 1.27 1.27)
+				)
+			)
+		)
+		(property "Datasheet" ""
+			(at 57.15 166.37 0)
+			(hide yes)
+			(show_name no)
+			(do_not_autoplace no)
+			(effects
+				(font
+					(size 1.27 1.27)
+				)
+			)
+		)
+		(property "Description" "Power symbol creates a global label with name \"+5V\""
+			(at 57.15 166.37 0)
+			(hide yes)
+			(show_name no)
+			(do_not_autoplace no)
+			(effects
+				(font
+					(size 1.27 1.27)
+				)
+			)
+		)
+		(pin "1"
+		)
+		(instances
+			(project "bled-stamp"
+				(path "/e988e766-358b-4d27-8746-3fe94b603f13"
+					(reference "#PWR096")
+					(unit 1)
+				)

Commit message: wip
Parts:
- removed TP1: TestPoint, symbol Connector:TestPoint
Connections:
- net PMIC_OTG: now reaches R19.1, U3.8 (OTG)
Changed lines of the file:
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@@
 	(wire
 		(pts
-			(xy 25.4 114.3) (xy 31.75 114.3)
+			(xy 27.94 114.3) (xy 31.75 114.3)
 		)
 		(stroke
@@
 		(property "Intersheetrefs" "${INTERSHEET_REFS}"
 			(at 46.8472 104.14 0)
+			(hide yes)
+			(show_name no)
+			(do_not_autoplace no)
+			(effects
+				(font
+					(size 1.27 1.27)
+				)
+				(justify right)
+			)
+		)
+	)
+	(global_label "PMIC_OTG"
+		(shape input)
+		(at 27.94 114.3 180)
+		(fields_autoplaced yes)
+		(effects
+			(font
+				(size 1.27 1.27)
+			)
+			(justify right)
+		)
+		(property "Intersheetrefs" "${INTERSHEET_REFS}"
+			(at 15.8229 114.3 0)
 			(hide yes)
 			(show_name no)
@@
 					(unit 1)
 				)
-			)
-		)
-	)
-	(symbol
-		(lib_id "Connector:TestPoint")
-		(at 25.4 114.3 90)
-		(unit 1)
-		(body_style 1)
-		(exclude_from_sim no)
-		(in_bom yes)
-		(on_board yes)
-		(in_pos_files yes)
-		(dnp no)
-		(fields_autoplaced yes)
-		(property "Reference" "TP1"
-			(at 22.098 109.22 90)
-			(show_name no)
-			(do_not_autoplace no)
-			(effects
-				(font
-					(size 1.27 1.27)
-				)
-			)
-		)
-		(property "Value" "TestPoint"
-			(at 22.098 111.76 90)
-			(show_name no)
-			(do_not_autoplace no)
-			(effects
-				(font
-					(size 1.27 1.27)
-				)
-			)
-		)
-		(property "Footprint" ""
-			(at 25.4 109.22 0)
-			(hide yes)
-			(show_name no)
-			(do_not_autoplace no)
-			(effects
-				(font
-					(size 1.27 1.27)
-				)
-			)
-		)
-		(property "Datasheet" ""
-			(at 25.4 109.22 0)
-			(hide yes)
-			(show_name no)
-			(do_not_autoplace no)
-			(effects
-				(font
-					(size 1.27 1.27)
-				)
-			)
-		)
-		(property "Description" "test point"
-			(at 25.4 114.3 0)
-			(hide yes)
-			(show_name no)
-			(do_not_autoplace no)
-			(effects
-				(font
-					(size 1.27 1.27)
-				)
-			)
-		)
-		(pin "1"
-		)
-		(instances
-			(project "bled-stamp"
-				(path "/e988e766-358b-4d27-8746-3fe94b603f13"
-					(reference "TP1")
-					(unit 1)
-				)
