File: pcb/bled-stamp/bled-stamp.kicad_pcb (KiCad board)
At the start: 2 copper layers, 29 parts, among them J4 TYPEC-304-ACP16, SW1 SW_Push, SW2 SW_Push, SW3 SW_Push, SW4 SW_Push, SW5 SW_Push, SW6 SW_Push, U1 RP2350A, U2 W25Q32RVXHJQ, U3 BQ25895RTWR, U4 TLV62595DMQR, U5 RM2, X1 ABM8-272-T3

Commit message: wip
Parts:
- added J6: Micro_SD_Card, bled:SD-Card-Deck-Hoauc-HYCW104-TF08-375B, F.Cu at (152.6, 65.3)
Connections:
- U3 pad 23: /Power/PMID -> +5V
- U3 pad 25: unconnected-(U3-PAD-Pad25) -> GND

Commit message: wip
Parts:
- added C10: 100n, Capacitor_SMD:C_0201_0603Metric, F.Cu at (172.8, 55.8)
- added C11: 100n, Capacitor_SMD:C_0201_0603Metric, F.Cu at (172.8, 57.5)
- added C12: 100n, Capacitor_SMD:C_0201_0603Metric, F.Cu at (172.8, 59.3)
- added C13: 100n, Capacitor_SMD:C_0201_0603Metric, F.Cu at (175.3, 50.5)
- added C14: 100n, Capacitor_SMD:C_0201_0603Metric, F.Cu at (175.3, 52.3)
- added C15: 100n, Capacitor_SMD:C_0201_0603Metric, F.Cu at (175.3, 54.0)
- added C16: 100n, Capacitor_SMD:C_0201_0603Metric, F.Cu at (175.3, 55.8)
- added C17: 4u7, Capacitor_SMD:C_0402_1005Metric, F.Cu at (185.3, 50.6)
- added C18: 4u7, Capacitor_SMD:C_0402_1005Metric, F.Cu at (185.3, 52.6)
- added C19: 4u7, Capacitor_SMD:C_0402_1005Metric, F.Cu at (185.3, 54.6)
- added C20: 4u7, Capacitor_SMD:C_0402_1005Metric, F.Cu at (185.3, 56.6)
- added C23: 4u7, Capacitor_SMD:C_0402_1005Metric, F.Cu at (185.3, 58.5)
- added C7: 100n, Capacitor_SMD:C_0201_0603Metric, F.Cu at (172.8, 50.5)
- added C8: 100n, Capacitor_SMD:C_0201_0603Metric, F.Cu at (172.8, 52.3)
- added C9: 100n, Capacitor_SMD:C_0201_0603Metric, F.Cu at (172.8, 54.0)
- added R10: 470R, Resistor_SMD:R_0201_0603Metric, F.Cu at (177.7, 55.8)
- added R11: 100R, Resistor_SMD:R_0201_0603Metric, F.Cu at (177.7, 57.5)
- added R12: 100R, Resistor_SMD:R_0201_0603Metric, F.Cu at (177.7, 59.3)
- added R13: 27R, Resistor_SMD:R_0201_0603Metric, F.Cu at (180.2, 50.5)
- added R14: 1K, Resistor_SMD:R_0201_0603Metric, F.Cu at (180.2, 52.3)
- added R15: 261R, Resistor_SMD:R_0201_0603Metric, F.Cu at (180.2, 54.0)
- added R16: 10k, Resistor_SMD:R_0201_0603Metric, F.Cu at (180.2, 55.8)
- added R17: 10k, Resistor_SMD:R_0201_0603Metric, F.Cu at (180.2, 57.5)
- added R18: 470R, Resistor_SMD:R_0201_0603Metric, F.Cu at (180.2, 59.3)
- added R19: 10k, Resistor_SMD:R_0201_0603Metric, F.Cu at (182.6, 50.5)
- added R20: 45k, Resistor_SMD:R_0201_0603Metric, F.Cu at (182.6, 52.3)
- added R21: 10k, Resistor_SMD:R_0201_0603Metric, F.Cu at (182.6, 54.0)
- added R22: 100k, Resistor_SMD:R_0201_0603Metric, F.Cu at (182.6, 55.8)
- added R23: 470R, Resistor_SMD:R_0201_0603Metric, F.Cu at (182.6, 57.5)
- added R24: 10k, Resistor_SMD:R_0201_0603Metric, F.Cu at (182.6, 59.3)
- added R5: 27R, Resistor_SMD:R_0201_0603Metric, F.Cu at (175.3, 57.5)
- added R6: 27R, Resistor_SMD:R_0201_0603Metric, F.Cu at (175.3, 59.3)
- added R7: 1k, Resistor_SMD:R_0201_0603Metric, F.Cu at (177.7, 50.5)
- added R8: 100R, Resistor_SMD:R_0201_0603Metric, F.Cu at (177.7, 52.3)
- added R9: 100R, Resistor_SMD:R_0201_0603Metric, F.Cu at (177.7, 54.0)
- added TP2: TestPoint, TestPoint:TestPoint_Pad_D1.0mm, F.Cu at (189.8, 89.7)
- moved J4 63.7 mm to (127.0, 108.0)
- moved U5 54.5 mm to (127.0, 69.8)
- moved J6 32.5 mm to (133.9, 91.9), turned to 90 degrees
- moved U3 24.6 mm to (190.1, 68.4)
- moved U2 19.6 mm to (185.6, 86.7)
- moved C39 16.7 mm to (188.7, 74.1)
- moved C6 16.7 mm to (188.7, 72.2)
- moved U4 15.8 mm to (190.7, 86.5)
- moved X1 8.15 mm to (180.4, 87.7)
- moved D3 7.61 mm to (175.1, 77.0)
- moved D4 7.61 mm to (175.1, 79.7)
- moved D5 7.61 mm to (175.1, 82.5)
- moved D6 7.61 mm to (175.1, 85.2)
- moved U1 4.56 mm to (181.2, 80.2)
- moved C40 1.64 mm to (189.5, 76.5)
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Connections:
- U3 pad 8: Net-(U3-OTG) -> PMIC_OTG
