File: pcb/bled-stamp/bled-stamp.kicad_pcb (KiCad board)
At the start: 2 copper layers, 68 parts, among them J4 TYPEC-304-ACP16, J6 Micro_SD_Card, SW1 SW_Push, SW2 SW_Push, SW3 SW_Push, SW4 SW_Push, SW5 SW_Push, SW6 SW_Push, U1 RP2350A, U2 W25Q32RVXHJQ, U3 BQ25895RTWR, U4 TLV62595DMQR, U5 RM2, X1 ABM8-272-T3

Commit message: wip
Parts:
- moved R19 24.8 mm to (187.3, 74.9)
- moved R20 24.8 mm to (187.3, 76.6)
- moved D3 24.5 mm to (195.3, 63.1)
- moved D4 24.5 mm to (195.3, 65.9)
- moved D5 24.5 mm to (195.3, 68.6)
- moved D6 24.5 mm to (195.3, 71.4)
- moved TP2 24.5 mm to (198.3, 66.8)
- moved C10 22.0 mm to (179.9, 76.6)
- moved C7 22.0 mm to (179.9, 71.4)
- moved C8 22.0 mm to (179.9, 73.1)
- moved C9 22.0 mm to (179.9, 74.9)
- moved L3 21.9 mm to (198.6, 63.5)
- moved L2 21.1 mm to (196.5, 85.7)
- moved R10 20.4 mm to (184.8, 74.9)
- moved R11 20.4 mm to (184.8, 76.6)
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