File: pcb/bled-stamp/bled-stamp.kicad_pcb (KiCad board)
At the start: 2 copper layers, 68 parts, among them J4 TYPEC-304-ACP16, J6 Micro_SD_Card, SW1 SW_Push, SW2 SW_Push, SW3 SW_Push, SW4 SW_Push, SW5 SW_Push, SW6 SW_Push, U1 RP2350A, U2 W25Q32RVXHJQ, U3 BQ25895RTWR, U4 TLV62595DMQR, U5 RM2, X1 ABM8-272-T3

Commit message: wip
Parts:
- added L1: AOTA-B201610S3R3-101-T, bled:IND_AOTA-B201610S_2p0x1p6x1p0_ABR-L, F.Cu at (184.2, 92.1)
Connections:
- U5 pad 13: WL_POWER -> BT_POWER
