File: pcb/bled-stamp/connectors.kicad_sch (KiCad schematic)
At the start: 9 parts, among them J1 Conn_01x12, J2 Conn_01x03, J3 Conn_01x02, J4 TYPEC-304-ACP16, J5 Conn_01x12, U5 RM2

Commit message: wip
Parts:
- R23, R24: footprint (none) -> Resistor_SMD:R_0201_0603Metric
Changed lines of the file:
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@@
 			)
 		)
-		(property "Footprint" ""
+		(property "Footprint" "Resistor_SMD:R_0201_0603Metric"
 			(at 54.61 160.528 90)
 			(hide yes)
@@
 			)
 		)
-		(property "Footprint" ""
+		(property "Footprint" "Resistor_SMD:R_0201_0603Metric"
 			(at 54.61 144.018 90)
 			(hide yes)
