File: pcb/bled-stamp/connectors.kicad_sch (KiCad schematic)
At the start: 9 parts, among them J1 Conn_01x12, J2 Conn_01x03, J3 Conn_01x02, J4 TYPEC-304-ACP16, J5 Conn_01x12, U5 RM2

Commit message: wip
Parts:
- removed C41: C, symbol Device:C
